Commit message: correct scale

File: src/curobo/content/assets/robot/iiwa_allegro_description/iiwa_virtuoso.urdf (robot description, URDF)
Before this commit: robot iiwa_virtuoso, 11 links, 10 joints
Links:
- link lbr_virtuoso: geometry collision mesh filename=/home/yanxi/curobo/src/curobo/content/assets/robot/iiwa_all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 scale=0.1 0.1 0.1; visual mesh filename=/home/yanxi/curobo/src/curobo/content/assets/robot/iiwa_all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 scale=0.1 0.1 0.1
Joints:
- removed joint lbr_joint_ee
- added joint lbr_joint_virtuoso: type fixed, parent lbr_link_7, child lbr_virtuoso, origin xyz=0 -0.28 0.11 rpy=1.57 0 0
- joint tool_tip_fixed_joint: origin xyz=0 0 0.1397 rpy=0 0 0 -> xyz=0 0 0.01397 rpy=0 0 0

Commit message: add kuka configs back for old kuka-virtuoso version

File: src/curobo/content/assets/robot/iiwa_allegro_description/iiwa_virtuoso.urdf (robot description, URDF)
Before this commit: robot iiwa_virtuoso, 11 links, 10 joints
Joints:
- joint lbr_world_joint: origin xyz=0 0 0 rpy=0 0 0 -> xyz=0 0 1.0 rpy=0 0 0
