Commit message: change robotiq gripper to a mesh

File: src/curobo/content/assets/robot/iiwa_allegro_description/iiwa_robotiq_test.urdf (robot description, URDF)
Before this commit: robot iiwa, 24 links, 23 joints
Links:
- removed link flange
- removed link left_inner_finger
- removed link left_inner_finger_pad
- removed link left_inner_knuckle
- removed link left_outer_finger
- removed link left_outer_knuckle
- removed link right_inner_finger
- removed link right_inner_finger_pad
- removed link right_inner_knuckle
- removed link right_outer_finger
- removed link right_outer_knuckle
- removed link robotiq_arg2f_base_link
- removed link tool0
- added link robotiq_base_link, mass 0.22652; collision mesh filename=/home/yanxi/curobo/src/curobo/content/assets/robot/iiwa_all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; visual mesh filename=/home/yanxi/curobo/src/curobo/content/assets/robot/iiwa_all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
- added link robotiq_to_iiwa_mount, mass 0.064; collision cylinder length=0.012 radius=0.035; visual cylinder length=0.012 radius=0.035
Joints:
- removed joint finger_joint
- removed joint flange-tool0
- removed joint gripper_base_joint
- removed joint left_inner_finger_joint
- removed joint left_inner_finger_pad_joint
- removed joint left_inner_knuckle_joint
- removed joint left_outer_finger_joint
- removed joint right_inner_finger_joint
- removed joint right_inner_finger_pad_joint
- removed joint right_inner_knuckle_joint
- removed joint right_outer_finger_joint
- removed joint right_outer_knuckle_joint
- removed joint wrist_3-flange
- added joint iiwa_to_mount: type fixed, parent iiwa_link_7, child robotiq_to_iiwa_mount, origin xyz=0 0 0.051 rpy=0 0 3.141592653589793
- added joint robotiq_mount_to_base_link: type fixed, parent robotiq_to_iiwa_mount, child robotiq_base_link, origin xyz=0 0 0.006 rpy=0 0 1.5708
- joint grasp_joint: parent robotiq_arg2f_base_link -> robotiq_to_iiwa_mount

Commit message: new left arm with color and configs

File: src/curobo/content/assets/robot/iiwa_allegro_description/iiwa_robotiq_test.urdf (robot description, URDF)
Before this commit: robot iiwa, 13 links, 12 joints
Links:
- removed link iiwa_link_0
- removed link iiwa_link_1
- removed link iiwa_link_2
- removed link iiwa_link_3
- removed link iiwa_link_4
- removed link iiwa_link_5
- removed link iiwa_link_6
- removed link iiwa_link_7
- removed link robot_table_link
- removed link robotiq_base_link
- removed link robotiq_to_iiwa_mount
- added link lbr_link_0, mass 7.050378; collision mesh filename=/home/yanxi/curobo/src/curobo/content/assets/robot/iiwa_all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; visual mesh filename=/home/yanxi/curobo/src/curobo/content/assets/robot/iiwa_all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
- added link lbr_link_1, mass 5.289529; collision mesh filename=/home/yanxi/curobo/src/curobo/content/assets/robot/iiwa_all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; visual mesh filename=/home/yanxi/curobo/src/curobo/content/assets/robot/iiwa_all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
- added link lbr_link_2, mass 5.688888; collision mesh filename=/home/yanxi/curobo/src/curobo/content/assets/robot/iiwa_all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; visual mesh filename=/home/yanxi/curobo/src/curobo/content/assets/robot/iiwa_all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
- added link lbr_link_3, mass 3.461245; collision mesh filename=/home/yanxi/curobo/src/curobo/content/assets/robot/iiwa_all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; visual mesh filename=/home/yanxi/curobo/src/curobo/content/assets/robot/iiwa_all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
- added link lbr_link_4, mass 4.122995; collision mesh filename=/home/yanxi/curobo/src/curobo/content/assets/robot/iiwa_all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; visual mesh filename=/home/yanxi/curobo/src/curobo/content/assets/robot/iiwa_all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
- added link lbr_link_5, mass 1.563756; collision mesh filename=/home/yanxi/curobo/src/curobo/content/assets/robot/iiwa_all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; visual mesh filename=/home/yanxi/curobo/src/curobo/content/assets/robot/iiwa_all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
- added link lbr_link_6, mass 2.457878; collision mesh filename=/home/yanxi/curobo/src/curobo/content/assets/robot/iiwa_all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; visual mesh filename=/home/yanxi/curobo/src/curobo/content/assets/robot/iiwa_all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
- added link lbr_link_7, mass 0.265331; collision mesh filename=/home/yanxi/curobo/src/curobo/content/assets/robot/iiwa_all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; visual mesh filename=/home/yanxi/curobo/src/curobo/content/assets/robot/iiwa_all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
- added link robotiq_link, mass 0.22652; collision mesh filename=/home/yanxi/curobo/src/curobo/content/assets/robot/iiwa_all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; visual mesh filename=/home/yanxi/curobo/src/curobo/content/assets/robot/iiwa_all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
- added link robotiq_to_lbr_mount, mass 0.064; collision mesh filename=/home/yanxi/curobo/src/curobo/content/assets/robot/iiwa_all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; visual mesh filename=/home/yanxi/curobo/src/curobo/content/assets/robot/iiwa_all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
Joints:
- removed joint iiwa_joint_1
- removed joint iiwa_joint_2
- removed joint iiwa_joint_3
- removed joint iiwa_joint_4
- removed joint iiwa_joint_5
- removed joint iiwa_joint_6
- removed joint iiwa_joint_7
- removed joint iiwa_to_mount
- removed joint robot_table_link_to_iiwa
- removed joint robotiq_mount_to_base_link
- removed joint world_to_right_table
- added joint lbr_A1: type revolute, parent lbr_link_0, child lbr_link_1, origin xyz=0.0 0.0 0.1475 rpy=0 0 0, axis 0.0 0.0 1.0, limit lower=-2.9670597283903604 upper=2.9670597283903604 effort=200 velocity=1.4835298641951802
- added joint lbr_A2: type revolute, parent lbr_link_1, child lbr_link_2, origin xyz=0.0 -0.01 0.2125 rpy=0 0 0, axis 0.0 1.0 0.0, limit lower=-2.0943951023931953 upper=2.0943951023931953 effort=200 velocity=1.4835298641951802
- added joint lbr_A3: type revolute, parent lbr_link_2, child lbr_link_3, origin xyz=0.0 0.01 0.228 rpy=0 0 0, axis 0.0 0.0 1.0, limit lower=-2.9670597283903604 upper=2.9670597283903604 effort=200 velocity=1.7453292519943295
- added joint lbr_A4: type revolute, parent lbr_link_3, child lbr_link_4, origin xyz=0.0 0.0105 0.192 rpy=0 0 0, axis 0.0 -1.0 0.0, limit lower=-2.0943951023931953 upper=2.0943951023931953 effort=200 velocity=1.3089969389957472
- added joint lbr_A5: type revolute, parent lbr_link_4, child lbr_link_5, origin xyz=0.0 -0.0105 0.2075 rpy=0 0 0, axis 0.0 0.0 1.0, limit lower=-2.9670597283903604 upper=2.9670597283903604 effort=200 velocity=2.2689280275926285
- added joint lbr_A6: type revolute, parent lbr_link_5, child lbr_link_6, origin xyz=0.0 -0.0707 0.1925 rpy=0 0 0, axis 0.0 1.0 0.0, limit lower=-2.0943951023931953 upper=2.0943951023931953 effort=200 velocity=2.356194490192345
- added joint lbr_A7: type revolute, parent lbr_link_6, child lbr_link_7, origin xyz=0.0 0.0707 0.091 rpy=0 0 0, axis 0.0 0.0 1.0, limit lower=-3.0543261909900763 upper=3.0543261909900763 effort=200 velocity=2.356194490192345
- added joint lbr_to_mount: type fixed, parent lbr_link_7, child robotiq_to_lbr_mount, origin xyz=0 0 0.0435 rpy=0 0 3.141592653589793
- added joint lbr_world_joint: type fixed, parent world, child lbr_link_0, origin xyz=0 0 0 rpy=0 0 3.14
- added joint mount_to_robotiq_link: type fixed, parent robotiq_to_lbr_mount, child robotiq_link, origin xyz=0 0 0.0056 rpy=0 0 0
- joint grasp_joint: parent robotiq_to_iiwa_mount -> robotiq_link

Commit message: rotate gripper mesh (not aligned with the usd)

File: src/curobo/content/assets/robot/iiwa_allegro_description/iiwa_robotiq_test.urdf (robot description, URDF)
Before this commit: robot iiwa_robotiq, 12 links, 11 joints
Joints:
- joint mount_to_robotiq_link: origin xyz=0 0 0.0056 rpy=0 0 0 -> xyz=0 0 0.0056 rpy=0 0 1.57
