Commit message: modified bimanual

File: src/curobo/content/assets/robot/iiwa_allegro_description/bimanual_iiwa_test.urdf (robot description, URDF)
Before this commit: robot bimanual, 43 links, 42 joints
Links:
- removed link left_lbr_link_ee
- removed link robotiq_grasp_frame
- added link grasp_frame, mass 0.01
- added link right_lbr_link_ee
Joints:
- removed joint left_lbr_joint_ee
- removed joint right_lbr_to_mount
- added joint lbr_to_mount: type fixed, parent left_lbr_link_7, child robotiq_to_lbr_mount, origin xyz=0 0 0.0435 rpy=0 0 3.141592653589793
- added joint right_lbr_joint_ee: type fixed, parent right_lbr_link_7, child right_lbr_link_ee, origin xyz=0 0 0.035 rpy=0 0 0
- joint grasp_joint: child robotiq_grasp_frame -> grasp_frame
- joint iiwa_to_mount: parent left_lbr_link_ee -> right_lbr_link_ee
- joint left_lbr_world_joint: origin xyz=0 0.45625 0 rpy=0 0 0 -> xyz=0 -0.45625 0 rpy=0 0 3.14
- joint mount_to_robotiq_link: origin xyz=0 0 0.0056 rpy=0 0 0 -> xyz=0 0 0.0056 rpy=0 0 1.57
- joint right_lbr_world_joint: origin xyz=0 -0.45625 0 rpy=0 0 3.14 -> xyz=0 0.45625 0 rpy=0 0 0
