Commit message: match the usd gripper orientation

File: src/curobo/content/assets/robot/iiwa_allegro_description/bimanual_robotiq.urdf (robot description, URDF)
Before this commit: robot bimanual, 21 links, 20 joints
Joints:
- joint right_mount_to_robotiq_link: origin xyz=0 0 0.0056 rpy=0 0 1.57 -> xyz=0 0 0.0056 rpy=0 0 -1.57
