Commit message: change to match the robot

File: src/curobo/content/assets/robot/iiwa_allegro_description/bimanual_robotiq_flat.urdf (robot description, URDF)
Before this commit: robot bimanual, 21 links, 20 joints
Joints:
- joint left_mount_to_robotiq_link: origin xyz=0 0 0.0056 rpy=0 0 1.57 -> xyz=0 0 0.0055 rpy=0 0 1.563756
- joint right_mount_to_robotiq_link: origin xyz=0 0 0.0056 rpy=0 0 -1.57 -> xyz=0 0 0.0055 rpy=0 0 -1.563756
